Commit message: mobile_robot gui, interfaces, core upload

File: mobile_robot_description/gazebo/mobile_robot.gazebo.xacro (robot description, xacro)
@@ -146,5 +146,5 @@
         </scan>
         <range>
-          <min>0.120</min>
+          <min>0.30</min>
           <max>10.5</max>
           <resolution>0.015</resolution>

File: mobile_robot_description/urdf/basic_mobile_robot.urdf (robot description, URDF)
Before this commit: robot mobile_robot, 3 links, 2 joints
Links:
- added link drivewhl_l_link; collision cylinder length=0.04 radius=0.10; visual cylinder length=0.04 radius=0.10
- added link drivewhl_r_link; collision cylinder length=0.04 radius=0.10; visual cylinder length=0.04 radius=0.10
- link base_link: geometry collision box size=0.42 0.31 0.09; visual box size=0.42 0.31 0.09
- link front_caster: geometry collision sphere radius=0.06; visual sphere radius=0.06
Joints:
- added joint drivewhl_l_joint: type continuous, parent base_link, child drivewhl_l_link, origin xyz=-0.12 0.18 -0.05 rpy=0 0 0, axis 0 1 0
- added joint drivewhl_r_joint: type continuous, parent base_link, child drivewhl_r_link, origin xyz=-0.12 -0.18 -0.05 rpy=0 0 0, axis 0 1 0
- joint base_joint: origin xyz=0.0 0.0 ${-(wheel_radius+wheel_zoff)} rpy=0 0 0 -> xyz=0.0 0.0 -0.15 rpy=0 0 0
- joint caster_joint: origin xyz=${caster_xoff} 0.0 ${-(base_height)} rpy=0 0 0 -> xyz=0.20 0.0 -0.09 rpy=0 0 0

File: mobile_robot_description/urdf/mobile_robot.urdf.xacro (robot description, xacro)
@@ -201,5 +201,3 @@
     <child link="camera_depth_frame"/>
   </joint>
-  <!-- Include gazebo macro -->
-  <xacro:include filename="$(find mobile_robot_description)/gazebo/mobile_robot.gazebo.xacro" />
 </robot>

File: mobile_robot_description/urdf/mobile_robot_gazebo.urdf.xacro (robot description, xacro)
@@ -202,4 +202,4 @@
   </joint>
   <!-- Include gazebo macro -->
-  <!-- <xacro:include filename="$(find mobile_robot_description)/gazebo/mobile_robot.gazebo.xacro" /> -->
+  <xacro:include filename="$(find mobile_robot_description)/gazebo/mobile_robot.gazebo.xacro" />
 </robot>
